Commit message: align bushing frames visually in rviz

File: models/2f_85_gripper/urdf/robotiq_85_gripper.urdf (robot description, URDF)
Before this commit: robot robotiq_85_gripper, 9 links, 8 joints
Links:
- added link left_bushing_A
- added link left_bushing_B
Joints:
- added joint test_A: type fixed, parent robotiq_85_left_finger_link, child left_bushing_A, origin xyz=0.047 -0.0057 0.0 rpy=0.0 0.0 0.0
- added joint test_B: type fixed, parent robotiq_85_left_finger_tip_link, child left_bushing_B, origin xyz=-0.007 -0.0174 0.0 rpy=0.0 0.0 0.0
